File: Embedded/AC_Logger/HW/PSU/PSU.kicad_sch (KiCad schematic)
At the start: 11 parts, among them T1 230V 3.2VA - 2x 12V 1.6VA, U1 L7809, U2 L7909

Commit message: Updated to new KiCAD version.
Parts:
- renumbered T1 to T?
