File: HW/Arduino_Automotive_Ultrasound_Shield_v1/Arduino_Automotive_Ultrasound_Shield_v1.kicad_pcb (KiCad board)
At the start: 2 copper layers, 9 parts, among them J1 Conn_01x04_Socket, J2 Conn_01x04_Socket, J3 Barrel_Jack_Switch, J4 Conn_01x04_Socket, J5 1x3 2.54mm male, J6 1x3 2.54mm male, SW1 SW_Push, U2 LM7805_TO220

Commit message: pcb
Parts:
- removed J4: Conn_01x04_Socket, Connector_PinSocket_2.54mm:PinSocket_1x04_P2.54mm_Vertical
- added H1: M3, MountingHole:MountingHole_3.2mm_M3, F.Cu at (86.4, 91.4)
- added H2: M3, MountingHole:MountingHole_3.2mm_M3, F.Cu at (157.5, 91.4)
- added H3: M3, MountingHole:MountingHole_3.2mm_M3, F.Cu at (86.4, 33.0)
- added H4: M3, MountingHole:MountingHole_3.2mm_M3, F.Cu at (157.5, 33.0)
- added J7: 1x4 2.54mm female, Connector_PinSocket_2.54mm:PinSocket_1x04_P2.54mm_Vertical, F.Cu at (121.9, 33.0)
- added SW2: SW_Push, Button_Switch_THT:SW_PUSH_6mm, F.Cu at (143.7, 76.2)
- added SW3: SW_Push, Button_Switch_THT:SW_PUSH_6mm, F.Cu at (153.8, 76.2)
- added SW4: SW_Push, Button_Switch_THT:SW_PUSH_6mm, F.Cu at (147.3, 78.7)
- J1, J2: value Conn_01x04_Socket -> 1x4 2.54mm female
- moved SW1 34.6 mm to (137.2, 78.7)
- moved U2 7.62 mm to (88.9, 83.8)
- moved J1 2.54 mm to (83.8, 58.4)
- moved J2 2.54 mm to (157.5, 53.3)
Connections:
- A2 pad 10: Net-(A2-D7) -> /ECHO_2
- A2 pad 16: unconnected-(A2-SCK-Pad16) -> /PB3
- A2 pad 19: /ECHO_0 -> /PB0
- A2 pad 20: /TRIG_0 -> /PB1
- A2 pad 21: unconnected-(A2-A2-Pad21) -> /PB2
- A2 pad 23: unconnected-(A2-SDA/A4-Pad23) -> /TRIG_1
- A2 pad 24: unconnected-(A2-SCL/A5-Pad24) -> /ECHO_1
- A2 pad 25: unconnected-(A2-A6-Pad25) -> /TRIG_0
- A2 pad 26: unconnected-(A2-A7-Pad26) -> /ECHO_0
- A2 pad 9: Net-(A2-D6) -> /TRIG_2
- J1 pad 1: (no net) -> GND
- J1 pad 2: (no net) -> /ECHO_2
- J1 pad 3: (no net) -> /TRIG_2
- J1 pad 4: (no net) -> +5V
- J2 pad 1: (no net) -> GND
- J2 pad 2: (no net) -> /ECHO_1
- J2 pad 3: (no net) -> /TRIG_1
- J2 pad 4: (no net) -> +5V
- SW1 pad 1: unconnected-(SW1-Pad1) -> /PB0
- SW1 pad 2: unconnected-(SW1-Pad2) -> GND
Routing:
- net GND: track 80.1 -> 255.8 mm, vias 4 -> 12
- net +5V: track 0.00 -> 114.3 mm, vias 0 -> 6
- net +12V: track 47.3 -> 98.8 mm, vias 2 -> 4
- net /TRIG_2: track 0.00 -> 50.8 mm, vias 0 -> 2
- net /ECHO_2: track 0.00 -> 50.8 mm, vias 0 -> 2
- net /PB3: track 0.00 -> 41.8 mm, vias 0 -> 2
- net /ECHO_1: track 0.00 -> 35.6 mm, vias 0 -> 2
- net /TRIG_1: track 0.00 -> 35.6 mm, vias 0 -> 2
- net /PB2: track 0.00 -> 17.6 mm
- net Vdrive: track 10.2 -> 17.8 mm
- net /PB1: track 0.00 -> 5.08 mm
- net /PB0: track 0.00 -> 5.08 mm
- net /ECHO_0: track 46.2 -> 45.7 mm, vias 0 -> 2
- net /TRIG_0: track 45.3 -> 45.7 mm, vias 0 -> 2
Other:
- board outline added: 81.3 x 68.6 mm

Commit message: promenjen pin
Connections:
- A2 pad 15: unconnected-(A2-MISO-Pad15) -> /PB3
- A2 pad 16: /PB3 -> unconnected-(A2-SCK-Pad16)
- A2 pad 19: /PB0 -> /PB2
- A2 pad 21: /PB2 -> /PB0
Routing:
- net /PB3: track 41.8 -> 62.1 mm

Commit message: test
Parts:
- moved J7 5.08 mm to (116.8, 33.0)
Connections:
- A2 pad 12: unconnected-(A2-D9-Pad12) -> /ECHO_0
- A2 pad 22: unconnected-(A2-A3-Pad22) -> /TRIG_0
- A2 pad 25: /TRIG_0 -> unconnected-(A2-A6-Pad25)
- A2 pad 26: /ECHO_0 -> unconnected-(A2-A7-Pad26)
Routing:
- net +5V: track 114.3 -> 119.4 mm
- net GND: track 255.8 -> 252.2 mm
- net /TRIG_0: track 45.7 -> 48.3 mm
- net /ECHO_0: track 45.7 -> 48.3 mm, vias 2 -> 1
Changed lines of the file:
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@@
 	(net 19 "+12V")
 	(net 20 "unconnected-(A2-~{RESET}-Pad3)")
-	(net 21 "unconnected-(A2-D9-Pad12)")
+	(net 21 "unconnected-(A2-A6-Pad25)")
 	(net 22 "Vdrive")
-	(net 23 "unconnected-(A2-A3-Pad22)")
+	(net 23 "unconnected-(A2-A7-Pad26)")
 	(net 24 "/TRIG_1")
 	(net 25 "/ECHO_1")
@@
 	(footprint "Connector_PinSocket_2.54mm:PinSocket_1x04_P2.54mm_Vertical"
 		(layer "F.Cu")
-		(at 121.92 33.02 90)
+		(at 116.84 33.02 90)
 		(descr "Through hole straight socket strip, 1x04, 2.54mm pitch, single row (from Kicad 4.0.7), script generated")
 		(tags "Through hole socket strip THT 1x04 2.54mm single row")
@@
 			)
 			(remove_unused_layers no)
-			(net 21 "unconnected-(A2-D9-Pad12)")
+			(net 4 "/ECHO_0")
 			(pinfunction "D9")
 			(pintype "bidirectional")
@@
 			)
 			(remove_unused_layers no)
-			(net 23 "unconnected-(A2-A3-Pad22)")
+			(net 17 "/TRIG_0")
 			(pinfunction "A3")
 			(pintype "bidirectional")
@@
 			)
 			(remove_unused_layers no)
-			(net 17 "/TRIG_0")
+			(net 21 "unconnected-(A2-A6-Pad25)")
 			(pinfunction "A6")
 			(pintype "bidirectional")
@@
 			)
 			(remove_unused_layers no)
-			(net 4 "/ECHO_0")
+			(net 23 "unconnected-(A2-A7-Pad26)")
 			(pinfunction "A7")
 			(pintype "bidirectional")
@@
 	)
 	(segment
+		(start 124.46 33.02)
+		(end 132.08 33.02)
+		(width 2)
+		(layer "B.Cu")
+		(net 2)
+	)
+	(segment
 		(start 132.08 58.42)
 		(end 127 58.42)
@@
 	)
 	(segment
-		(start 129.54 33.02)
-		(end 132.08 33.02)
-		(width 2)
-		(layer "B.Cu")
-		(net 2)
-	)
-	(segment
 		(start 132.08 58.42)
 		(end 139.7 58.42)
@@
 	)
 	(segment
-		(start 114.3 81.28)
-		(end 114.3 91.44)
-		(width 2)
-		(layer "F.Cu")
-		(net 3)
-	)
-	(segment
 		(start 114.3 33.02)
 		(end 114.3 58.42)
@@
 	)
 	(segment
-		(start 111.76 58.42)
-		(end 111.76 81.28)
+		(start 109.22 58.42)
+		(end 109.22 81.28)
+		(width 2)
+		(layer "F.Cu")
+		(net 3)
+	)
+	(segment
+		(start 96.52 91.44)
+		(end 96.52 81.28)
 		(width 2)
 		(layer "F.Cu")
@@
 	)
 	(via
-		(at 111.76 58.42)
+		(at 96.52 81.28)
+		(size 2)
+		(drill 1)
+		(layers "F.Cu" "B.Cu")
+		(net 3)
+	)
+	(via
+		(at 109.22 58.42)
 		(size 2)
 		(drill 1)
@@
 	)
 	(via
-		(at 114.3 81.28)
+		(at 96.52 91.44)
 		(size 2)
 		(drill 1)
@@
 	)
 	(via
-		(at 114.3 91.44)
+		(at 109.22 81.28)
 		(size 2)
 		(drill 1)
@@
 		(net 3)
 	)
-	(via
-		(at 111.76 81.28)
-		(size 2)
-		(drill 1)
-		(layers "F.Cu" "B.Cu")
+	(segment
+		(start 107.4225 92.36)
+		(end 110.4225 89.36)
+		(width 2)
+		(layer "B.Cu")
 		(net 3)
 	)
@@
 	)
 	(segment
-		(start 114.3 91.44)
-		(end 106.6425 91.44)
+		(start 132.08 53.34)
+		(end 157.48 53.34)
 		(width 2)
 		(layer "B.Cu")
@@
 	)
 	(segment
-		(start 132.08 53.34)
-		(end 157.48 53.34)
+		(start 104.8025 91.44)
+		(end 105.7225 92.36)
+		(width 2)
+		(layer "B.Cu")
+		(net 3)
+	)
+	(segment
+		(start 96.52 91.44)
+		(end 104.8025 91.44)
+		(width 2)
+		(layer "B.Cu")
+		(net 3)
+	)
+	(segment
+		(start 106.68 81.28)
+		(end 109.22 81.28)
 		(width 2)
 		(layer "B.Cu")
@@
 	)
 	(segment
-		(start 106.68 81.28)
-		(end 114.3 81.28)
+		(start 116.84 58.42)
+		(end 121.92 58.42)
 		(width 2)
 		(layer "B.Cu")
@@
 	)
 	(segment
-		(start 116.84 58.42)
-		(end 121.92 58.42)
+		(start 156.9 71.7)
+		(end 157.48 71.12)
 		(width 2)
 		(layer "B.Cu")
@@
 	)
 	(segment
-		(start 156.9 71.7)
-		(end 157.48 71.12)
+		(start 116.84 33.02)
+		(end 114.3 33.02)
 		(width 2)
 		(layer "B.Cu")
@@
 	)
 	(segment
-		(start 106.6425 91.44)
-		(end 105.7225 92.36)
+		(start 105.7225 92.36)
+		(end 107.4225 92.36)
 		(width 2)
 		(layer "B.Cu")
@@
 	)
 	(segment
-		(start 121.92 33.02)
-		(end 114.3 33.02)
-		(width 2)
-		(layer "B.Cu")
-		(net 3)
-	)
-	(segment
-		(start 134.62 60.96)
-		(end 134.62 30.48)
+		(start 119.38 78.74)
+		(end 119.38 33.02)
 		(width 2)
 		(layer "F.Cu")
@@
 	)
 	(via
-		(at 134.62 60.96)
-		(size 2)
-		(drill 1)
-		(layers "F.Cu" "B.Cu")
-		(net 4)
-	)
-	(via
-		(at 134.62 30.48)
+		(at 119.38 78.74)
 		(size 2)
 		(drill 1)
@@
 	)
 	(segment
-		(start 124.46 33.02)
-		(end 124.46 30.48)
-		(width 2)
-		(layer "B.Cu")
-		(net 4)
-	)
-	(segment
-		(start 132.08 60.96)
-		(end 134.62 60.96)
-		(width 2)
-		(layer "B.Cu")
-		(net 4)
-	)
-	(segment
-		(start 124.46 30.48)
-		(end 134.62 30.48)
+		(start 119.38 78.74)
+		(end 116.84 78.74)
 		(width 2)
 		(layer "B.Cu")
@@
 	)
 	(segment
-		(start 137.16 35.56)
-		(end 137.16 63.5)
+		(start 129.54 35.56)
+		(end 129.54 71.12)
 		(width 2)
 		(layer "F.Cu")
@@
 	)
 	(via
-		(at 137.16 35.56)
+		(at 129.54 71.12)
 		(size 2)
 		(drill 1)
@@
 	)
 	(via
-		(at 137.16 63.5)
+		(at 129.54 35.56)
 		(size 2)
 		(drill 1)
@@
 	)
 	(segment
-		(start 137.16 63.5)
-		(end 132.08 63.5)
+		(start 129.54 71.12)
+		(end 132.08 71.12)
 		(width 2)
 		(layer "B.Cu")
@@
 	)
 	(segment
-		(start 127 35.56)
-		(end 137.16 35.56)
+		(start 121.92 35.56)
+		(end 129.54 35.56)
 		(width 2)
 		(layer "B.Cu")
@@
 	)
 	(segment
-		(start 127 35.56)
-		(end 127 33.02)
+		(start 121.92 33.02)
+		(end 121.92 35.56)
 		(width 2)
 		(layer "B.Cu")
